Commit message: rotate laser scanner 90 degree clock-wise

File: urdf/includes/pablowsky_simplified_model.xacro (robot description, xacro)
@@ -114,5 +114,5 @@
     <parent link="base_link"/>
     <child link="base_scan"/>
-    <origin xyz="-0.032 0 0.172" rpy="0 0 0"/>
+    <origin xyz="-0.032 0 0.172" rpy="0 0 -1.5708"/>
   </joint>
   <link name="base_scan">

Commit message: rotate lidar 180 degrees to match real robot

File: urdf/includes/pablowsky_simplified_model.xacro (robot description, xacro)
@@ -114,5 +114,5 @@
     <parent link="base_link"/>
     <child link="base_scan"/>
-    <origin xyz="-0.032 0 0.172" rpy="0 0 -1.5708"/>
+    <origin xyz="-0.032 0 0.172" rpy="0 0 1.5708"/>
   </joint>
   <link name="base_scan">
